File: hw/746-hfp-kicad/746-hfp-kicad.kicad_sch (KiCad schematic)
At the start: 47 parts, among them J1 Conn_01x01_Socket, J10 Conn_01x01_Socket, J11 Conn_01x01_Socket, J12 Conn_01x12_Socket, J13 Conn_01x01_Socket, J14 Conn_01x01_Socket, J15 Conn_01x01_Socket, J16 Conn_01x01_Socket, J17 Conn_01x01_Socket, J18 Conn_01x01_Socket, J19 Conn_01x01_Socket, J2 Conn_01x01_Socket, J20 Conn_01x01_Socket, J21 Conn_01x01_Socket, J22 Conn_01x01_Socket, J23 Conn_01x01_Socket, J24 Conn_01x01_Socket, J25 Conn_01x01_Socket, J26 Conn_01x01_Socket, J27 Conn_01x01_Socket, J3 Conn_01x01_Socket, J4 Conn_01x01_Socket, J5 Conn_01x01_Socket, J6 Conn_01x01_Socket, J7 Conn_01x01_Socket, J8 Conn_01x01_Socket, J9 Conn_01x01_Socket, Q1 NMOS, U1 UA741, U2 Pico, U4 LM358

Commit message: Bug fixes
Parts:
- R3: value 100k -> 20k
Changed lines of the file:
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@@
   (symbol (lib_id "Device:R") (at 103.0732 33.3756 90) (unit 1)
     (in_bom yes) (on_board yes) (dnp no) (fields_autoplaced)
-    (property "Reference" "R3" (at 103.0732 27.7368 90)
+    (property "Reference" "R3" (at 103.0732 27.94 90)
       (effects (font (size 1.27 1.27)))
     )
-    (property "Value" "100k" (at 103.0732 30.2768 90)
+    (property "Value" "20k" (at 103.0732 30.48 90)
       (effects (font (size 1.27 1.27)))
     )

Commit message: WIP
Parts:
- added J28: Conn_01x01_Socket, symbol Connector:Conn_01x01_Socket
Connections:
- net ADC_RX (27): now reaches U2.16 (GPIO12)
- net ADC_TX_In (27) renamed ADC_TX (27)
- new net ADC_RX (26): J28.1 (Pin_1)
Changed lines of the file:
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@@
   (junction (at 172.6184 57.15) (diameter 0) (color 0 0 0 0)
   )
-  (wire (pts (xy 176.276 60.9092) (xy 169.2656 60.9092))
+  (wire (pts (xy 176.276 58.166) (xy 165.7096 58.166))
     (stroke (width 0) (type default))
   )
@@
     (stroke (width 0) (type default))
   )
+  (wire (pts (xy 166.2176 61.468) (xy 180.0352 61.468))
+    (stroke (width 0) (type default))
+  )
   (wire (pts (xy 244.9576 147.9296) (xy 247.65 147.9296))
     (stroke (width 0) (type default))
@@
     (stroke (width 0) (type default))
   )
-  (wire (pts (xy 170.2308 57.15) (xy 172.6184 57.15))
+  (wire (pts (xy 168.3004 57.15) (xy 172.6184 57.15))
     (stroke (width 0) (type default))
   )
@@
     (stroke (width 0) (type default))
   )
-  (wire (pts (xy 170.2308 57.3024) (xy 170.2308 57.15))
+  (wire (pts (xy 168.3004 55.372) (xy 168.3004 57.15))
     (stroke (width 0) (type default))
   )
@@
     (stroke (width 0) (type default))
   )
+  (wire (pts (xy 180.0352 61.468) (xy 180.0352 60.452))
+    (stroke (width 0) (type default))
+  )
   (wire (pts (xy 182.8292 57.912) (xy 176.276 57.912))
     (stroke (width 0) (type default))
@@
     (stroke (width 0) (type default))
   )
-  (wire (pts (xy 176.276 57.912) (xy 176.276 60.9092))
+  (wire (pts (xy 176.276 57.912) (xy 176.276 58.166))
     (stroke (width 0) (type default))
   )
@@
   )
   (wire (pts (xy 223.2152 65.532) (xy 218.3892 65.532))
+    (stroke (width 0) (type default))
+  )
+  (wire (pts (xy 180.0352 60.452) (xy 182.8292 60.452))
     (stroke (width 0) (type default))
   )
@@
     )
   )
+  (global_label "ADC_RX (27)" (shape input) (at 166.2176 61.468 180) (fields_autoplaced)
+    (effects (font (size 1.27 1.27)) (justify right))
+    (property "Intersheetrefs" "${INTERSHEET_REFS}" (at 151.0767 61.468 0)
+      (effects (font (size 1.27 1.27)) (justify right) hide)
+    )
+  )
   (global_label "5Vin" (shape input) (at 91.3384 43.4848 90) (fields_autoplaced)
     (effects (font (size 1.27 1.27)) (justify left))
@@
     )
   )
-  (global_label "ADC_TX_In (27)" (shape output) (at 169.2656 60.9092 180) (fields_autoplaced)
-    (effects (font (size 1.27 1.27)) (justify right))
-    (property "Intersheetrefs" "${INTERSHEET_REFS}" (at 151.7057 60.9092 0)
+  (global_label "ADC_TX (27)" (shape output) (at 165.7096 58.166 180) (fields_autoplaced)
+    (effects (font (size 1.27 1.27)) (justify right))
+    (property "Intersheetrefs" "${INTERSHEET_REFS}" (at 150.8711 58.166 0)
       (effects (font (size 1.27 1.27)) (justify right) hide)
     )
@@
     )
   )
-  (global_label "ADC_TX_In (27)" (shape input) (at 40.1828 80.0608 180) (fields_autoplaced)
-    (effects (font (size 1.27 1.27)) (justify right))
-    (property "Intersheetrefs" "${INTERSHEET_REFS}" (at 22.6229 80.0608 0)
-      (effects (font (size 1.27 1.27)) (justify right) hide)
-    )
-  )
-  (global_label "ADC_SLCK (12)" (shape output) (at 170.2308 57.3024 180) (fields_autoplaced)
-    (effects (font (size 1.27 1.27)) (justify right))
-    (property "Intersheetrefs" "${INTERSHEET_REFS}" (at 152.7918 57.3024 0)
+  (global_label "ADC_TX (27)" (shape input) (at 40.1828 80.0608 180) (fields_autoplaced)
+    (effects (font (size 1.27 1.27)) (justify right))
+    (property "Intersheetrefs" "${INTERSHEET_REFS}" (at 25.3443 80.0608 0)
+      (effects (font (size 1.27 1.27)) (justify right) hide)
+    )
+  )
+  (global_label "ADC_SLCK (12)" (shape output) (at 168.3004 55.372 180) (fields_autoplaced)
+    (effects (font (size 1.27 1.27)) (justify right))
+    (property "Intersheetrefs" "${INTERSHEET_REFS}" (at 150.8614 55.372 0)
       (effects (font (size 1.27 1.27)) (justify right) hide)
     )
@@
     (effects (font (size 1.27 1.27)) (justify right))
     (property "Intersheetrefs" "${INTERSHEET_REFS}" (at 24.829 56.7944 0)
+      (effects (font (size 1.27 1.27)) (justify right) hide)
+    )
+  )
+  (global_label "ADC_RX (26)" (shape output) (at 39.9796 84.582 180) (fields_autoplaced)
+    (effects (font (size 1.27 1.27)) (justify right))
+    (property "Intersheetrefs" "${INTERSHEET_REFS}" (at 24.8387 84.582 0)
       (effects (font (size 1.27 1.27)) (justify right) hide)
     )
@@
         )
       )
+    )
+  )
+  (symbol (lib_name "Conn_01x01_Socket_3") (lib_id "Connector:Conn_01x01_Socket") (at 45.0596 84.582 0) (unit 1)
+    (in_bom yes) (on_board yes) (dnp no) (fields_autoplaced)
+    (property "Reference" "J28" (at 45.8216 83.312 0)
+      (effects (font (size 1.27 1.27)) (justify left))
+    )
+    (property "Value" "Conn_01x01_Socket" (at 45.8216 85.852 0)
+      (effects (font (size 1.27 1.27)) (justify left))
+    )
+    (property "Footprint" "" (at 45.0596 84.582 0)
+      (effects (font (size 1.27 1.27)) hide)
+    )
+    (property "Datasheet" "~" (at 45.0596 84.582 0)
+      (effects (font (size 1.27 1.27)) hide)
+    )
+    (pin "1")
+    (instances
+      (project "746-hfp-kicad"
+        (path "/a73d1afc-f0a5-418c-8247-1028a7b305b8"
+          (reference "J28") (unit 1)
+        )
+      )

Commit message: WIP
Parts:
- removed J21, J22, J23, J26: Conn_01x01_Socket, symbol Connector:Conn_01x01_Socket
- added C8: 10uF, symbol Device:C
- added R4: 1k, symbol Device:R
- RV2: value 10k (6.7k to Mic+) -> 10k
Connections:
- net ADC_CS (14) is gone; now on net Audio_SCL (14): J25.1 (Pin_1)
- net ADC_RX (27) is gone; now on net Audio_SDA (26): U2.16 (GPIO12)
- net DAC_CS (5) is gone; now on net DAC_CS (17): J10.1 (Pin_1)
- net DAC_TX_Din (23) is gone; now on net DAC_TX_Din (19): J5.1 (Pin_1)
- net 3.3Vin_Clean: now also R4.1; no longer RV2.2
- net ADC_In: now also C8.2; no longer J12.3 (Pin_3), RV2.1
- net AGND: now also RV2.1
- net DAC_SCLK (18): now also U2.24 (GPIO18)
- net Audio_SCL (14): now reaches U2.17 (GPIO13)
- net DAC_CS (17): now reaches U2.22 (GPIO17)
- net DAC_TX_Din (19): now reaches U2.25 (GPIO19)
- net ADC_Enable (13) renamed Audio_Enable (13)
- net ADC_RX (26) renamed Audio_SDA (26)
- net ADC_SLCK (12): no longer names the net of U2.14 (GPIO10)
- net ADC_TX (27): no longer names the net of U2.15 (GPIO11)
- net ADC_TX (27): no longer J24.1 (Pin_1)
- new net Audio_Ready (25): J24.1 (Pin_1)
- new net Mic+: C8.1, J12.3 (Pin_3), R4.2
Other:
- note added: "50/50"
- moved on the sheet: C2, C5, C6, C7, J25, J27, J28, R3, U2, U4A, U4B, U4C

Commit message: Stable(ish)
Parts:
- added R5: 330, symbol Device:R
- added R6: 100k, symbol Device:R
- added RV3: 100k, symbol Device:R_Potentiometer_Trim
- added U3: TL431P, Package_DIP:DIP-8_W7.62mm, symbol Reference_Voltage:TL431P
Connections:
- net 3.3Vin_Clean: no longer R4.1
- net 5Vin: now also R5.1
- net AGND: now also U3.6 (A)
- new net: R5.2, RV3.1, U3.1 (K)
- new net: R6.1, RV3.3
Changed lines of the file:
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@@
   (junction (at 98.3488 104.8512) (diameter 0) (color 0 0 0 0)
   )
+  (junction (at 83.7692 91.44) (diameter 0) (color 0 0 0 0)
+  )
   (junction (at 130.302 26.1112) (diameter 0) (color 0 0 0 0)
   )
+  (junction (at 73.4568 97.4344) (diameter 0) (color 0 0 0 0)
+  )
   (junction (at 92.7608 23.5204) (diameter 0) (color 0 0 0 0)
   )
@@
   (junction (at 55.626 135.5852) (diameter 0) (color 0 0 0 0)
   )
+  (junction (at 73.1012 84.6836) (diameter 0) (color 0 0 0 0)
+  )
   (junction (at 207.4164 34.8488) (diameter 0) (color 0 0 0 0)
   )
@@
     (stroke (width 0) (type default))
   )
+  (wire (pts (xy 73.4568 105.0544) (xy 83.7184 105.0544))
+    (stroke (width 0) (type default))
+  )
   (wire (pts (xy 244.9576 147.9296) (xy 247.65 147.9296))
     (stroke (width 0) (type default))
   )
+  (wire (pts (xy 83.7692 84.6836) (xy 83.7692 91.44))
+    (stroke (width 0) (type default))
+  )
   (wire (pts (xy 265.1252 149.1996) (xy 262.636 149.1996))
     (stroke (width 0) (type default))
@@
     (stroke (width 0) (type default))
   )
+  (wire (pts (xy 83.7692 91.44) (xy 98.298 91.44))
+    (stroke (width 0) (type default))
+  )
   (wire (pts (xy 165.8112 65.3288) (xy 171.8564 65.3288))
     (stroke (width 0) (type default))
   )
+  (wire (pts (xy 81.28 90.5764) (xy 81.28 93.98))
+    (stroke (width 0) (type default))
+  )
   (wire (pts (xy 92.7608 23.5204) (xy 92.7608 27.178))
     (stroke (width 0) (type default))
@@
     (stroke (width 0) (type default))
   )
+  (wire (pts (xy 83.7692 96.52) (xy 83.7692 108.8136))
+    (stroke (width 0) (type default))
+  )
   (wire (pts (xy 278.13 150.7236) (xy 270.256 150.7236))
     (stroke (width 0) (type default))
@@
     (stroke (width 0) (type default))
   )
+  (wire (pts (xy 73.1012 83.4136) (xy 73.1012 84.6836))
+    (stroke (width 0) (type default))
+  )
   (wire (pts (xy 210.82 60.5536) (xy 210.82 60.452))
     (stroke (width 0) (type default))
   )
+  (wire (pts (xy 76.9112 90.5764) (xy 81.28 90.5764))
+    (stroke (width 0) (type default))
+  )
   (wire (pts (xy 95.4024 104.8512) (xy 98.3488 104.8512))
     (stroke (width 0) (type default))
@@
     (stroke (width 0) (type default))
   )
+  (wire (pts (xy 83.7184 105.0544) (xy 83.7184 105.0036))
+    (stroke (width 0) (type default))
+  )
   (wire (pts (xy 55.9816 128.6002) (xy 43.5356 128.6002))
     (stroke (width 0) (type default))
@@
     (stroke (width 0) (type default))
   )
+  (wire (pts (xy 73.1012 94.3864) (xy 73.1012 95.7072))
+    (stroke (width 0) (type default))
+  )
+  (wire (pts (xy 73.1012 84.6836) (xy 73.1012 86.7664))
+    (stroke (width 0) (type default))
+  )
   (wire (pts (xy 98.2472 157.48) (xy 98.1964 157.48))
     (stroke (width 0) (type default))
   )
+  (wire (pts (xy 73.1012 95.7072) (xy 73.5076 95.7072))
+    (stroke (width 0) (type default))
+  )
   (wire (pts (xy 46.7106 162.3822) (xy 48.7426 162.3822))
     (stroke (width 0) (type default))
@@
     (stroke (width 0) (type default))
   )
+  (wire (pts (xy 73.152 73.4568) (xy 73.152 75.7936))
+    (stroke (width 0) (type default))
+  )
   (wire (pts (xy 100.4316 32.7152) (xy 116.7384 32.7152))
     (stroke (width 0) (type default))
   )
+  (wire (pts (xy 73.4568 97.4344) (xy 73.5076 97.4344))
+    (stroke (width 0) (type default))
+  )
   (wire (pts (xy 167.132 50.038) (xy 167.132 46.5328))
     (stroke (width 0) (type default))
@@
     (stroke (width 0) (type default))
   )
+  (wire (pts (xy 73.5076 95.7072) (xy 73.5076 97.4344))
+    (stroke (width 0) (type default))
+  )
+  (wire (pts (xy 73.1012 84.6836) (xy 83.7692 84.6836))
+    (stroke (width 0) (type default))
+  )
   (wire (pts (xy 91.5924 23.5204) (xy 92.7608 23.5204))
     (stroke (width 0) (type default))
@@
     (stroke (width 0) (type default))
   )
+  (wire (pts (xy 73.152 75.7936) (xy 73.1012 75.7936))
+    (stroke (width 0) (type default))
+  )
+  (wire (pts (xy 73.406 97.4344) (xy 73.4568 97.4344))
+    (stroke (width 0) (type default))
+  )
   (wire (pts (xy 270.002 147.1676) (xy 270.002 149.7076))
     (stroke (width 0) (type default))
@@
     (fill (type none))
   )
-  (rectangle (start 87.5792 75.946) (end 146.4564 116.5352)
+  (rectangle (start 69.2404 64.77) (end 146.4564 116.5352)
     (stroke (width 0) (type default))
     (fill (type none))
@@
     )
   )
+  (global_label "AGND" (shape output) (at 83.7692 108.8136 270) (fields_autoplaced)
+    (effects (font (size 1.27 1.27)) (justify right))
+    (property "Intersheetrefs" "${INTERSHEET_REFS}" (at 83.7692 116.7579 90)
+      (effects (font (size 1.27 1.27)) (justify right) hide)
+    )
+  )
   (global_label "Mic+" (shape output) (at 240.538 141.0716 90) (fields_autoplaced)
     (effects (font (size 1.27 1.27) (color 0 0 255 1)) (justify left))
@@
     )
   )
-  (global_label "3.3Vin_Clean" (shape input) (at 98.3488 91.2368 90) (fields_autoplaced)
-    (effects (font (size 1.27 1.27)) (justify left))
-    (property "Intersheetrefs" "${INTERSHEET_REFS}" (at 98.3488 76.096 90)
-      (effects (font (size 1.27 1.27)) (justify left) hide)
-    )
-  )
   (global_label "GND" (shape output) (at 212.2424 67.8688 0) (fields_autoplaced)
     (effects (font (size 1.27 1.27)) (justify left))
@@
     )
   )
+  (global_label "5Vin" (shape input) (at 73.152 73.4568 90) (fields_autoplaced)
+    (effects (font (size 1.27 1.27)) (justify left))
+    (property "Intersheetrefs" "${INTERSHEET_REFS}" (at 73.152 66.4197 90)
+      (effects (font (size 1.27 1.27)) (justify left) hide)
+    )
+  )
   (global_label "DAC_TX_Din (19)" (shape input) (at 252.7808 71.6788 180) (fields_autoplaced)
     (effects (font (size 1.27 1.27)) (justify right))
@@
     )
   )
+  (symbol (lib_id "Reference_Voltage:TL431P") (at 83.7692 93.98 90) (unit 1)
+    (in_bom yes) (on_board yes) (dnp no) (fields_autoplaced)
+    (property "Reference" "U3" (at 86.1568 92.71 90)
+      (effects (font (size 1.27 1.27)) (justify right))
+    )
+    (property "Value" "TL431P" (at 86.1568 95.25 90)
+      (effects (font (size 1.27 1.27)) (justify right))
+    )
+    (property "Footprint" "Package_DIP:DIP-8_W7.62mm" (at 87.5792 93.98 0)
+      (effects (font (size 1.27 1.27) italic) hide)
+    )
+    (property "Datasheet" "http://www.ti.com/lit/ds/symlink/tl431.pdf" (at 83.7692 93.98 0)
+      (effects (font (size 1.27 1.27) italic) hide)
+    )
+    (pin "1")
+    (pin "6")
+    (pin "8")
+    (instances
+      (project "746-hfp-kicad"
+        (path "/a73d1afc-f0a5-418c-8247-1028a7b305b8"
+          (reference "U3") (unit 1)
+        )
+      )
+    )
+  )
   (symbol (lib_id "Device:C") (at 234.3912 60.5028 0) (unit 1)
     (in_bom yes) (on_board yes) (dnp no) (fields_autoplaced)
@@
         (path "/a73d1afc-f0a5-418c-8247-1028a7b305b8"
           (reference "J11") (unit 1)
+        )
+      )
+    )
+  )
+  (symbol (lib_id "Device:R") (at 73.4568 101.2444 0) (unit 1)
+    (in_bom yes) (on_board yes) (dnp no) (fields_autoplaced)
+    (property "Reference" "R6" (at 76.1492 99.9744 0)
+      (effects (font (size 1.27 1.27)) (justify left))
+    )
+    (property "Value" "100k" (at 76.1492 102.5144 0)
+      (effects (font (size 1.27 1.27)) (justify left))
+    )
+    (property "Footprint" "" (at 71.6788 101.2444 90)
+      (effects (font (size 1.27 1.27)) hide)
+    )
+    (property "Datasheet" "~" (at 73.4568 101.2444 0)
+      (effects (font (size 1.27 1.27)) hide)
+    )
+    (pin "1")
+    (pin "2")
+    (instances
+      (project "746-hfp-kicad"
+        (path "/a73d1afc-f0a5-418c-8247-1028a7b305b8"
+          (reference "R6") (unit 1)
         )
       )
@@
     )
   )
+  (symbol (lib_id "Device:R_Potentiometer_Trim") (at 73.1012 90.5764 0) (unit 1)
+    (in_bom yes) (on_board yes) (dnp no) (fields_autoplaced)
+    (property "Reference" "RV3" (at 70.9676 89.3064 0)
+      (effects (font (size 1.27 1.27)) (justify right))
+    )
+    (property "Value" "100k" (at 70.9676 91.8464 0)
+      (effects (font (size 1.27 1.27)) (justify right))
+    )
+    (property "Footprint" "" (at 73.1012 90.5764 0)
+      (effects (font (size 1.27 1.27)) hide)
+    )
+    (property "Datasheet" "~" (at 73.1012 90.5764 0)
+      (effects (font (size 1.27 1.27)) hide)
+    )
+    (pin "1")
+    (pin "2")
+    (pin "3")
+    (instances
+      (project "746-hfp-kicad"
+        (path "/a73d1afc-f0a5-418c-8247-1028a7b305b8"
+          (reference "RV3") (unit 1)
+        )
+      )
+    )
+  )
   (symbol (lib_id "Amplifier_Operational:LM358") (at 117.0432 40.64 0) (unit 2)
     (in_bom yes) (on_board yes) (dnp no)
@@
         )
       )
+    )
+  )
+  (symbol (lib_id "Device:R") (at 73.1012 79.6036 0) (unit 1)
+    (in_bom yes) (on_board yes) (dnp no) (fields_autoplaced)
+    (property "Reference" "R5" (at 78.9432 79.6036 90)
+      (effects (font (size 1.27 1.27)))
+    )
+    (property "Value" "330" (at 76.4032 79.6036 90)
+      (effects (font (size 1.27 1.27)))
+    )
+    (property "Footprint" "" (at 71.3232 79.6036 90)
+      (effects (font (size 1.27 1.27)) hide)
+    )
+    (property "Datasheet" "~" (at 73.1012 79.6036 0)
+      (effects (font (size 1.27 1.27)) hide)
+    )
+    (pin "1")
+    (pin "2")
+    (instances
+      (project "746-hfp-kicad"
+        (path "/a73d1afc-f0a5-418c-8247-1028a7b305b8"
+          (reference "R5") (unit 1)
+        )
+      )
