File: hw/746-hfp-kicad/746-hfp-kicad.kicad_sch (KiCad schematic)
At the start: 50 parts, among them J1 Conn_01x01_Socket, J10 Conn_01x01_Socket, J11 Conn_01x01_Socket, J12 Conn_01x12_Socket, J13 Conn_01x01_Socket, J14 Conn_01x01_Socket, J15 Conn_01x01_Socket, J16 Conn_01x01_Socket, J17 Conn_01x01_Socket, J18 Conn_01x01_Socket, J19 Conn_01x01_Socket, J2 Conn_01x01_Socket, J20 Conn_01x01_Socket, J24 Conn_01x01_Socket, J25 Conn_01x01_Socket, J27 Conn_01x01_Socket, J28 Conn_01x01_Socket, J3 Conn_01x01_Socket, J4 Conn_01x01_Socket, J5 Conn_01x01_Socket, J6 Conn_01x01_Socket, J7 Conn_01x01_Socket, J8 Conn_01x01_Socket, J9 Conn_01x01_Socket, Q1 NMOS, U1 UA741, U2 Pico, U3 TL431P, U4 LM358

Commit message: WIP
Parts:
- added C9: 0.1uF, symbol Device:C
Connections:
- net 3.3Vin_Clean: now also R5.2, RV3.1, U2.35 (ADC_VREF), U3.1 (K); no longer U2.36 (3V3)
- net ADC_In: now also U2.31 (GPIO26_ADC0), C9.2; no longer U2.32 (GPIO27_ADC1)
- net AGND: now also C9.1
Changed lines of the file:
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@@
   (junction (at 116.7384 26.0604) (diameter 0) (color 0 0 0 0)
   )
-  (junction (at 210.7692 34.8488) (diameter 0) (color 0 0 0 0)
-  )
-  (junction (at 210.7184 34.8488) (diameter 0) (color 0 0 0 0)
-  )
   (junction (at 98.3488 104.8512) (diameter 0) (color 0 0 0 0)
   )
@@
   (junction (at 92.7608 23.5204) (diameter 0) (color 0 0 0 0)
   )
+  (junction (at 213.868 50.4444) (diameter 0) (color 0 0 0 0)
+  )
+  (junction (at 83.7692 84.6836) (diameter 0) (color 0 0 0 0)
+  )
   (junction (at 53.3146 162.3822) (diameter 0) (color 0 0 0 0)
   )
@@
   (junction (at 73.1012 84.6836) (diameter 0) (color 0 0 0 0)
   )
-  (junction (at 207.4164 34.8488) (diameter 0) (color 0 0 0 0)
-  )
   (junction (at 127.1524 92.5576) (diameter 0) (color 0 0 0 0)
   )
-  (wire (pts (xy 210.7692 34.8488) (xy 210.7692 34.8996))
+  (junction (at 213.868 38.6588) (diameter 0) (color 0 0 0 0)
+  )
+  (wire (pts (xy 207.4164 37.3888) (xy 209.1944 37.3888))
     (stroke (width 0) (type default))
   )
@@
     (stroke (width 0) (type default))
   )
+  (wire (pts (xy 86.5632 84.6836) (xy 86.5632 85.0392))
+    (stroke (width 0) (type default))
+  )
   (wire (pts (xy 39.8272 33.3248) (xy 39.3192 33.3248))
     (stroke (width 0) (type default))
@@
     (stroke (width 0) (type default))
   )
-  (wire (pts (xy 210.7184 34.798) (xy 210.7692 34.798))
-    (stroke (width 0) (type default))
-  )
   (wire (pts (xy 40.1828 24.384) (xy 39.6748 24.384))
     (stroke (width 0) (type default))
@@
     (stroke (width 0) (type default))
   )
+  (wire (pts (xy 207.4164 47.5488) (xy 208.534 47.5488))
+    (stroke (width 0) (type default))
+  )
   (wire (pts (xy 53.3146 162.3822) (xy 53.3146 166.1922))
     (stroke (width 0) (type default))
@@
     (stroke (width 0) (type default))
   )
+  (wire (pts (xy 210.9724 38.6588) (xy 213.868 38.6588))
+    (stroke (width 0) (type default))
+  )
   (wire (pts (xy 247.65 150.2156) (xy 249.936 150.2156))
     (stroke (width 0) (type default))
@@
     (stroke (width 0) (type default))
   )
-  (wire (pts (xy 210.7184 34.8488) (xy 210.7184 34.798))
-    (stroke (width 0) (type default))
-  )
   (wire (pts (xy 46.7106 162.3822) (xy 46.7106 175.5902))
     (stroke (width 0) (type default))
@@
     (stroke (width 0) (type default))
   )
+  (wire (pts (xy 213.868 50.4444) (xy 208.534 50.4444))
+    (stroke (width 0) (type default))
+  )
   (wire (pts (xy 273.7612 113.792) (xy 270.256 113.792))
     (stroke (width 0) (type default))
@@
     (stroke (width 0) (type default))
   )
+  (wire (pts (xy 213.868 38.6588) (xy 213.868 40.5892))
+    (stroke (width 0) (type default))
+  )
   (wire (pts (xy 249.936 150.2156) (xy 249.936 150.7236))
     (stroke (width 0) (type default))
@@
     (stroke (width 0) (type default))
   )
-  (wire (pts (xy 207.4164 45.0088) (xy 211.9376 45.0088))
-    (stroke (width 0) (type default))
-  )
   (wire (pts (xy 168.91 52.6288) (xy 168.91 50.546))
     (stroke (width 0) (type default))
@@
     (stroke (width 0) (type default))
   )
+  (wire (pts (xy 83.7692 84.6836) (xy 86.5632 84.6836))
+    (stroke (width 0) (type default))
+  )
   (wire (pts (xy 210.0072 65.3288) (xy 210.0072 64.3128))
     (stroke (width 0) (type default))
@@
     (stroke (width 0) (type default))
   )
+  (wire (pts (xy 208.534 50.4444) (xy 208.534 47.5488))
+    (stroke (width 0) (type default))
+  )
   (wire (pts (xy 72.4916 153.3652) (xy 72.4408 153.3652))
     (stroke (width 0) (type default))
@@
     (stroke (width 0) (type default))
   )
-  (wire (pts (xy 207.4164 34.798) (xy 207.4164 34.8488))
-    (stroke (width 0) (type default))
-  )
   (wire (pts (xy 250.444 150.7236) (xy 250.444 149.4536))
     (stroke (width 0) (type default))
   )
+  (wire (pts (xy 213.868 38.6588) (xy 217.7288 38.6588))
+    (stroke (width 0) (type default))
+  )
   (wire (pts (xy 73.5076 95.7072) (xy 73.5076 97.4344))
     (stroke (width 0) (type default))
   )
+  (wire (pts (xy 209.1944 34.798) (xy 210.7692 34.798))
+    (stroke (width 0) (type default))
+  )
   (wire (pts (xy 73.1012 84.6836) (xy 83.7692 84.6836))
     (stroke (width 0) (type default))
@@
     (stroke (width 0) (type default))
   )
+  (wire (pts (xy 86.5632 85.0392) (xy 87.7316 85.0392))
+    (stroke (width 0) (type default))
+  )
   (wire (pts (xy 165.8112 65.3288) (xy 165.8112 64.1604))
     (stroke (width 0) (type default))
@@
     (stroke (width 0) (type default))
   )
-  (wire (pts (xy 207.4164 34.8488) (xy 210.7184 34.8488))
-    (stroke (width 0) (type default))
-  )
   (wire (pts (xy 207.4164 62.7888) (xy 209.296 62.7888))
     (stroke (width 0) (type default))
@@
     (stroke (width 0) (type default))
   )
-  (wire (pts (xy 210.7184 34.8488) (xy 210.7692 34.8488))
-    (stroke (width 0) (type default))
-  )
   (wire (pts (xy 122.0724 92.6084) (xy 127.1524 92.5576))
     (stroke (width 0) (type default))
@@
     (stroke (width 0) (type default))
   )
+  (wire (pts (xy 209.1944 37.3888) (xy 209.1944 34.798))
+    (stroke (width 0) (type default))
+  )
   (wire (pts (xy 211.2772 31.2928) (xy 211.2772 29.7688))
     (stroke (width 0) (type default))
@@
     (stroke (width 0) (type default))
   )
-  (wire (pts (xy 210.9724 38.6588) (xy 212.852 38.6588))
+  (wire (pts (xy 215.4428 50.4444) (xy 213.868 50.4444))
     (stroke (width 0) (type default))
   )
@@
     (stroke (width 0) (type default))
   )
-  (wire (pts (xy 210.7692 34.798) (xy 210.7692 34.8488))
-    (stroke (width 0) (type default))
-  )
   (wire (pts (xy 247.65 150.2156) (xy 247.65 147.9296))
     (stroke (width 0) (type default))
@@
     (stroke (width 0) (type default))
   )
+  (wire (pts (xy 217.7288 38.6588) (xy 217.7288 38.608))
+    (stroke (width 0) (type default))
+  )
   (wire (pts (xy 163.2204 54.9148) (xy 163.9824 54.9148))
+    (stroke (width 0) (type default))
+  )
+  (wire (pts (xy 213.868 48.2092) (xy 213.868 50.4444))
     (stroke (width 0) (type default))
   )
@@
     )
   )
-  (global_label "3.3Vin_Clean" (shape output) (at 210.7184 34.798 0) (fields_autoplaced)
-    (effects (font (size 1.27 1.27)) (justify left))
-    (property "Intersheetrefs" "${INTERSHEET_REFS}" (at 225.8592 34.798 0)
+  (global_label "3.3Vin_Clean" (shape output) (at 87.7316 85.0392 0) (fields_autoplaced)
+    (effects (font (size 1.27 1.27)) (justify left))
+    (property "Intersheetrefs" "${INTERSHEET_REFS}" (at 102.8724 85.0392 0)
       (effects (font (size 1.27 1.27)) (justify left) hide)
     )
@@
     )
   )
-  (global_label "ADC_In" (shape input) (at 211.9376 45.0088 0) (fields_autoplaced)
-    (effects (font (size 1.27 1.27)) (justify left))
-    (property "Intersheetrefs" "${INTERSHEET_REFS}" (at 221.2728 45.0088 0)
+  (global_label "ADC_In" (shape input) (at 215.4428 50.4444 0) (fields_autoplaced)
+    (effects (font (size 1.27 1.27)) (justify left))
+    (property "Intersheetrefs" "${INTERSHEET_REFS}" (at 224.778 50.4444 0)
       (effects (font (size 1.27 1.27)) (justify left) hide)
     )
@@
     )
   )
-  (global_label "AGND" (shape output) (at 212.852 38.6588 0) (fields_autoplaced)
-    (effects (font (size 1.27 1.27)) (justify left))
-    (property "Intersheetrefs" "${INTERSHEET_REFS}" (at 220.7963 38.6588 0)
+  (global_label "AGND" (shape output) (at 217.7288 38.6588 0) (fields_autoplaced)
+    (effects (font (size 1.27 1.27)) (justify left))
+    (property "Intersheetrefs" "${INTERSHEET_REFS}" (at 225.6731 38.6588 0)
       (effects (font (size 1.27 1.27)) (justify left) hide)
     )
@@
     (effects (font (size 1.27 1.27) (color 118 56 0 1)) (justify left))
     (property "Intersheetrefs" "${INTERSHEET_REFS}" (at 254 128.4586 90)
+      (effects (font (size 1.27 1.27)) (justify left) hide)
+    )
+  )
+  (global_label "3.3Vin_Clean" (shape input) (at 210.7692 34.798 0) (fields_autoplaced)
+    (effects (font (size 1.27 1.27)) (justify left))
+    (property "Intersheetrefs" "${INTERSHEET_REFS}" (at 225.91 34.798 0)
       (effects (font (size 1.27 1.27)) (justify left) hide)
     )
@@
         )
       )
+    )
+  )
+  (symbol (lib_id "Device:C") (at 213.868 44.3992 0) (unit 1)
+    (in_bom yes) (on_board yes) (dnp no) (fields_autoplaced)
+    (property "Reference" "C9" (at 218.0336 43.1292 0)
+      (effects (font (size 1.27 1.27)) (justify left))
+    )
+    (property "Value" "0.1uF" (at 218.0336 45.6692 0)
+      (effects (font (size 1.27 1.27)) (justify left))
+    )
+    (property "Footprint" "" (at 214.8332 48.2092 0)
+      (effects (font (size 1.27 1.27)) hide)
+    )
+    (property "Datasheet" "~" (at 213.868 44.3992 0)
+      (effects (font (size 1.27 1.27)) hide)
+    )
+    (pin "1")
+    (pin "2")
+    (instances
+      (project "746-hfp-kicad"
+        (path "/a73d1afc-f0a5-418c-8247-1028a7b305b8"
+          (reference "C9") (unit 1)
+        )
+      )

Commit message: Update schematic
Parts:
- removed unit 2 of U1
- added C10: 220uF, symbol Device:C
- added R7: 10k, symbol Device:R
Connections:
- net 5Vin: now also C10.1, R7.2
- net AGND: now also C4.2
- net GND: now also C10.2; no longer C4.2
Other:
- moved on the sheet: D4, J12, R2

Commit message: Update schematic
Parts:
- added C11: 220uF, symbol Device:C
- added D5, D6: LED, symbol Device:LED
- added J21, J22: Conn_01x01_Socket, symbol Connector:Conn_01x01_Socket
- added R8: 2k, symbol Device:R
- added R9: 1k, symbol Device:R
- added SW1: SW_Push, symbol Switch:SW_Push
- added SW2: SW_SPST, symbol Switch:SW_SPST
Connections:
- net 3.3Vin: now also SW1.1
- net 5Vin: now also SW2.1 (A); no longer C1.1
- net GND: now also C1.1, C11.1, R8.2, R9.2; no longer C1.2
- new net: D6.1 (K), R9.1
- new net: C1.2, C11.2, D6.2 (A), SW2.2 (B)
- new net: D5.1 (K), R8.1
- new net BT_LED_STATE (19): D5.2 (A), J22.1 (Pin_1)
- new net ENABLE_PAIRING_BTN (18): J21.1 (Pin_1), SW1.2
Other:
- note added: "Blue"
- note added: "Bluetooth connection control & state LED indicator"
- note added: "Red"
- moved on the sheet: C1

Commit message: Update schematic
Parts:
- C1, C2, C4, C6, C7, C8, C9: footprint (none) -> Capacitor_THT:C_Disc_D4.7mm_W2.5mm_P5.00mm
- C10, C11, C3, C5: footprint (none) -> Capacitor_THT:C_Radial_D6.3mm_H11.0mm_P2.50mm
- D1, D2: footprint (none) -> Diode_THT:D_DO-41_SOD81_P10.16mm_Horizontal
- D3, D4, D5, D6: footprint (none) -> LED_THT:LED_D5.0mm
- J1, J10, J11, J12, J13, J14, J15, J16, J17, J18, J19, J2, J20, J21, J22, J24, J25, J27, J28, J3, J4, J5, J6, J7, J8, J9: footprint (none) -> Connector_PinHeader_2.54mm:PinHeader_1x01_P2.54mm_Vertical
- Q1: footprint (none) -> Package_TO_SOT_THT:TO-220-3_Vertical
- R1, R2, R3, R4, R5, R6, R7, R8, R9: footprint (none) -> Resistor_THT:R_Axial_DIN0207_L6.3mm_D2.5mm_P10.16mm_Horizontal
- RV1: footprint (none) -> Potentiometer_THT:Potentiometer_Runtron_RM-065_Vertical
- RV2, RV3: footprint (none) -> Potentiometer_THT:Potentiometer_Bourns_3296W_Vertical
- SW1: footprint (none) -> Button_Switch_THT:SW_PUSH_6mm_H5mm
- SW2: footprint (none) -> Connector_PinHeader_2.54mm:PinHeader_1x02_P2.54mm_Vertical
- U1, U4: footprint (none) -> Package_DIP:DIP-8_W7.62mm_Socket_LongPads
- U3: footprint Package_DIP:DIP-8_W7.62mm -> Package_TO_SOT_THT:TO-92_Inline_Wide
