File: hw/746-hfp-kicad/746-hfp-kicad.kicad_sch (KiCad schematic)
At the start: 62 parts, among them J1 Conn_01x01_Socket, J10 Conn_01x01_Socket, J11 Conn_01x01_Socket, J12 Conn_01x12_Socket, J13 Conn_01x01_Socket, J14 Conn_01x01_Socket, J15 Conn_01x01_Socket, J16 Conn_01x01_Socket, J17 Conn_01x01_Socket, J18 Conn_01x01_Socket, J19 Conn_01x01_Socket, J2 Conn_01x01_Socket, J20 Conn_01x01_Socket, J21 Conn_01x01_Socket, J22 Conn_01x01_Socket, J24 Conn_01x01_Socket, J25 Conn_01x01_Socket, J27 Conn_01x01_Socket, J28 Conn_01x01_Socket, J3 Conn_01x01_Socket, J4 Conn_01x01_Socket, J5 Conn_01x01_Socket, J6 Conn_01x01_Socket, J7 Conn_01x01_Socket, J8 Conn_01x01_Socket, J9 Conn_01x01_Socket, Q1 NMOS, SW1 SW_Push, SW2 SW_SPST, U1 UA741, U2 Pico, U3 TL431P, U4 LM358

Commit message: Improve schematic
Parts:
- removed C7: 0.1uf, Capacitor_THT:C_Disc_D4.7mm_W2.5mm_P5.00mm, symbol Device:C
- removed J13, J14, J15, J16, J17, J18, J19, J20, J21, J22, J24, J25, J27, J28: Conn_01x01_Socket, Connector_PinHeader_2.54mm:PinHeader_1x01_P2.54mm_Vertical, symbol Connector:Conn_01x01_Socket
- removed SW1: SW_Push, Button_Switch_THT:SW_PUSH_6mm_H5mm, symbol Switch:SW_Push
- added C12: 220uF, Capacitor_THT:C_Radial_D6.3mm_H11.0mm_P2.50mm, symbol Device:C
- added C13: 0.1uf, Capacitor_THT:C_Disc_D4.7mm_W2.5mm_P5.00mm, symbol Device:C
- added J13, J14: Conn_01x15_Pin, Connector_PinHeader_2.54mm:PinHeader_1x15_P2.54mm_Vertical, symbol Connector:Conn_01x15_Pin
- added J15: Conn_01x02, symbol Connector_Generic:Conn_01x02
- added SW3: SW_Push, Button_Switch_THT:SW_PUSH_6mm_H5mm, symbol Switch:SW_Push
- C10: value 220uF -> 0.1uF
- C4: value 0.1uf -> 220uF
- D1, D2: value D_Schottky -> 1N5819
- Q1: value NMOS -> IRFZ44N
Connections:
- net 33Vout is gone; now on net 34Vout: U1.8 (V+)
- net ADC_In is gone; now on an unnamed net: C8.2, C9.2, U2.31 (GPIO26_ADC0)
- net AGND is gone; now on net GNDA: C4.2, C6.1, C9.1, J12.2 (Pin_2), J12.4 (Pin_4), J7.1 (Pin_1), RV2.1, U2.33 (AGND), U3.6 (A), U4.4 (V-), U4.5 (+)
- net 3.3Vin: now also J14.15 (Pin_15), SW3.2
- net 3.3Vin_Clean: now also R4.1, RV2.3
- net 5Vin: now also C10.2, C2.2, R7.1, C12.2, C13.1; no longer C10.1, C2.1, R7.2, SW2.1 (A)
- net Audio_SCL (14): now also J13.11 (Pin_11)
- net Audio_SDA (26): now also J13.9 (Pin_9)
- net BT_LED_STATE (19): now also J14.6 (Pin_6)
- net DOut: now also R7.2
- net Dialer (15): now also J14.13 (Pin_13)
- net ENABLE_PAIRING_BTN (18): now also J14.7 (Pin_7), SW3.1
- net GND: now also C2.1, U2.42 (GND), C12.1, J13.14 (Pin_14), J14.14 (Pin_14), J15.2 (Pin_2); no longer C10.2, C2.2
- net HookSwitchOut (2): now also J14.12 (Pin_12)
- net HookSwitchPower (4): now also J14.11 (Pin_11)
- net RingerEnabled (17): now also J14.9 (Pin_9)
- net RingerSignal (16): now also J14.10 (Pin_10)
- net at Q1.1 (D), U1.4 (V-): now also D2.1 (K)
- net at U3.8 (REF): now also RV3.2
- net GNDA: now reaches R6.2
- net GNDA: now also C10.1, C13.2
- net at C1.2, C11.2, D6.2 (A)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: now also J13.15 (Pin_15)
- net at C5.1, U4.1: now also U4.2 (-)
- net Pico_Enable: now reaches U2.37 (3V3_EN)
- net Pico_Enable: now also J13.1 (Pin_1)
- net Audio_Enable (13): no longer names the net of U2.12 (GPIO9)
- new net +5V: J15.1 (Pin_1), SW2.1 (A)
Other:
- note added: "Bluetooth connection state LED indicator"
- note removed: "Bluetooth connection control & state LED indicator"
- company: (none) -> Vlad Balmos
- title: (none) -> GPO-746-Bluetooth-conversion
- moved on the sheet: C1, C10, C11, C2, C3, C4, C5, C6, C8, C9, D1, D2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

Commit message: Improved schematic
Parts:
- removed U1: UA741, Package_DIP:DIP-8_W7.62mm_Socket_LongPads, symbol Device:Opamp_Dual
- added U5: UA741, symbol Simulation_SPICE:OPAMP
Connections:
- net 34Vout: now also U5.7 (V+)
- net GND: now also R6.2, RV2.1, U3.6 (A); no longer U2.42 (GND)
- net GNDA: no longer R6.2, RV2.1, U3.6 (A)
- net RingerSignal (16): now also U5.3 (+)
- net Mosfet_Drain: now reaches D2.1 (K), Q1.1 (D)
- net Mosfet_Drain: now also U5.4 (V-)
- net at C3.2, D1.1 (K), RV1.3: now also U5.6
- net at RV1.2: now also U5.2 (-)
Other:
- moved on the sheet: C1, C10, C11, C12, C13, C2, C3, C4, C5, C6, C8, C9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

Commit message: Generate bill of materials
Parts:
- J15: footprint (none) -> Connector_PinHeader_2.54mm:PinHeader_1x15_P2.54mm_Vertical
- U5: footprint (none) -> Package_DIP:DIP-8_W7.62mm_Socket_LongPads
Changed lines of the file:
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@@
       (effects (font (size 1.27 1.27)))
     )
-    (property "Footprint" "" (at 205.74 99.06 0)
+    (property "Footprint" "Package_DIP:DIP-8_W7.62mm_Socket_LongPads" (at 205.74 99.06 0)
       (effects (font (size 1.27 1.27)) hide)
     )
@@
       (effects (font (size 1.27 1.27)) (justify left))
     )
-    (property "Footprint" "" (at 39.37 217.17 0)
-      (effects (font (size 1.27 1.27)) hide)
-    )
+    (property "Footprint" "Connector_PinHeader_2.54mm:PinHeader_1x15_P2.54mm_Vertical" (at 39.37 217.17 0)
+      (effects (font (size 1.27 1.27)) hide)
+    )

Commit message: Improve schematic
Parts:
- removed D3, D4, D6: LED, LED_THT:LED_D5.0mm, symbol Device:LED
- removed R1, R2: 220, Resistor_THT:R_Axial_DIN0207_L6.3mm_D2.5mm_P10.16mm_Horizontal, symbol Device:R
- removed R9: 1k, Resistor_THT:R_Axial_DIN0207_L6.3mm_D2.5mm_P10.16mm_Horizontal, symbol Device:R
- removed SW2: SW_SPST, Connector_PinHeader_2.54mm:PinHeader_1x02_P2.54mm_Vertical, symbol Switch:SW_SPST
- removed SW3: SW_Push, Button_Switch_THT:SW_PUSH_6mm_H5mm, symbol Switch:SW_Push
- added J17: Control_board_connector, Connector_JST:JST_PH_B8B-PH-K_1x08_P2.00mm_Vertical, symbol Connector:Conn_01x08_Pin
- J1: value Conn_01x01_Socket -> 5V
- J12: value Conn_01x12_Socket -> Phone_Connector
- J13: value Conn_01x15_Pin -> ESP32_Left_Pins
- J14: value Conn_01x15_Pin -> ESP32_Right_Pins
- J15: value Conn_01x02 -> Power_Connector
- J2, J4: value Conn_01x01_Socket -> GND
- J3: value Conn_01x01_Socket -> 34V
- U2: footprint RPi_Pico:RPi_Pico_SMD_TH -> MCU_RaspberryPi_and_Boards:RPi_Pico_SMD_TH
Connections:
- net 5Vin is gone; now on net +5V: C10.2, C12.2, C13.1, C2.2, C4.1, J1.1 (Pin_1), J8.1 (Pin_1), R5.1, R7.1, U2.39 (VSYS), U4.8 (V+)
- net +5V: now also C1.2, C11.2, J13.15 (Pin_15); no longer J15.1 (Pin_1)
- net BT_LED_STATE (19): now also J17.4 (Pin_4)
- net ENABLE_PAIRING_BTN (18): now also J17.3 (Pin_3)
- net GND: now also J17.8 (Pin_8)
- net HookSwitchOut (2): now also J17.6 (Pin_6)
- net RingerSignal (16): now also J17.5 (Pin_5)
- net 3.3Vin renamed +3.3V
- net +3.3V: now also J17.2 (Pin_2)
- net 3.3Vin_Clean renamed +3.3V_Clean
- net 34Vout renamed +34V
- new net +5V_pre_switch: J15.1 (Pin_1), J17.1 (Pin_1)
Other:
- added sheet Control board (GPO-746-bt-control-board.kicad_sch)
- note added: "Connector to control board"
- note removed: "Green"
- note removed: "Headset off-hook visual indicator"
- note removed: "Red"
- note removed: "Yellow"
- title: GPO-746-Bluetooth-conversion -> GPO-746-Bluetooth-conversion Main board

Commit message: Create pcb board
Parts:
- removed D5: LED, LED_THT:LED_D5.0mm, symbol Device:LED
- removed R8: 2k, Resistor_THT:R_Axial_DIN0207_L6.3mm_D2.5mm_P10.16mm_Horizontal, symbol Device:R
- added J18: Conn_01x01_Socket, Connector_PinSocket_2.54mm:PinSocket_1x01_P2.54mm_Vertical, symbol Connector:Conn_01x01_Socket
- C11, C12: symbol Device:C -> Device:C_Polarized
- C4: footprint Capacitor_THT:C_Disc_D4.7mm_W2.5mm_P5.00mm -> Capacitor_THT:C_Radial_D6.3mm_H11.0mm_P2.50mm; symbol Device:C -> Device:C_Polarized
- J1, J10, J11, J2, J3, J4, J5, J6, J7, J8, J9: footprint Connector_PinHeader_2.54mm:PinHeader_1x01_P2.54mm_Vertical -> Connector_PinSocket_2.54mm:PinSocket_1x01_P2.54mm_Vertical
- J12: footprint Connector_PinHeader_2.54mm:PinHeader_1x01_P2.54mm_Vertical -> Connector_PinSocket_2.54mm:PinSocket_1x12_P2.54mm_Vertical
- J13, J14: footprint Connector_PinHeader_2.54mm:PinHeader_1x15_P2.54mm_Vertical -> Connector_PinSocket_2.54mm:PinSocket_1x15_P2.54mm_Vertical
- J15: footprint Connector_PinHeader_2.54mm:PinHeader_1x15_P2.54mm_Vertical -> Connector_PinHeader_2.54mm:PinHeader_1x02_P2.54mm_Vertical
- RV1: value 100k - 14k (to gnd) 80k (to output) -> 100k
Connections:
- net +5V: now also C11.1, C12.1, J17.7 (Pin_7); no longer C11.2, C12.2
- net GND: now also C11.2, C12.2; no longer C11.1, C12.1
- net Pico_Enable: now also U2.30 (RUN); no longer U2.37 (3V3_EN)
- net Audio_SCL (27): now reaches J13.8 (Pin_8)
- net Audio_SCL (27): now also U2.17 (GPIO13)
- net Audio_SCL (14): no longer names the net of J13.11 (Pin_11)
- net Audio_SCL (14): no longer U2.17 (GPIO13)
Other:
- note added: "1 - 2: 20k; 2 - 3: 80k"
- note added: "Tune RV2 to bias the Mic to 1.65v"
- note added: "Tune RV3 in order to get 3.3V from the regulator"
- note removed: "50/50"
- note removed: "Blue"
- note removed: "Bluetooth connection state LED indicator"
- moved on the sheet: C6, R3
