File: hw/746-hfp-kicad/GPO-746-bt-control-board.kicad_sch (KiCad schematic)
At the start: 11 parts, among them J16 Control_board_Connector, SW1 SW_Push, SW4 SW_SPST

Commit message: Create pcb board
Parts:
- J16: footprint Connector_PinHeader_2.54mm:PinHeader_1x08_P2.54mm_Vertical -> Connector_PinSocket_2.54mm:PinSocket_1x15_P2.54mm_Vertical
Connections:
- net +5V: now also J16.7 (Pin_7)
Changed lines of the file:
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@@
   (junction (at 203.2 109.22) (diameter 0) (color 0 0 0 0)
   )
+  (wire (pts (xy 99.06 58.42) (xy 99.06 81.28))
+    (stroke (width 0) (type default))
+  )
   (wire (pts (xy 93.98 73.66) (xy 134.62 73.66))
     (stroke (width 0) (type default))
@@
     (stroke (width 0) (type default))
   )
+  (wire (pts (xy 93.98 81.28) (xy 99.06 81.28))
+    (stroke (width 0) (type default))
+  )
   (wire (pts (xy 160.02 109.22) (xy 203.2 109.22))
     (stroke (width 0) (type default))
@@
     (stroke (width 0) (type default))
   )
+  (wire (pts (xy 99.06 58.42) (xy 203.2 58.42))
+    (stroke (width 0) (type default))
+  )
   (wire (pts (xy 93.98 78.74) (xy 129.54 78.74))
     (stroke (width 0) (type default))
@@
   )
   (wire (pts (xy 93.98 76.2) (xy 132.08 76.2))
+    (stroke (width 0) (type default))
+  )
+  (wire (pts (xy 203.2 58.42) (xy 203.2 66.04))
     (stroke (width 0) (type default))
   )
@@
       (effects (font (size 1.27 1.27)) (justify left))
     )
-    (property "Footprint" "Connector_PinHeader_2.54mm:PinHeader_1x08_P2.54mm_Vertical" (at 88.9 73.66 0)
-      (effects (font (size 1.27 1.27)) hide)
-    )
+    (property "Footprint" "Connector_PinSocket_2.54mm:PinSocket_1x15_P2.54mm_Vertical" (at 88.9 73.66 0)
+      (effects (font (size 1.27 1.27)) hide)
+    )
